Commit message: to run planning on irb120

File: catkin_ws/src/pnpush_config/models/IRB120/irb_120.urdf (robot description, URDF)
Before this commit: robot irb_120, 7 links, 6 joints
Links:
- link base_link: geometry collision mesh filename=package://pnpush_config/models/IRB120/meshes/collision/base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 scale=0.0254 0.0254 0.0254; visual mesh filename=package://pnpush_config/models/IRB120/meshes/visual/base_li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 scale=0.0254 0.0254 0.0254
- link link_1: geometry collision mesh filename=package://pnpush_config/models/IRB120/meshes/collision/link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 scale=0.0254 0.0254 0.0254; visual mesh filename=package://pnpush_config/models/IRB120/meshes/visual/link_1.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 scale=0.0254 0.0254 0.0254
- link link_2: geometry collision mesh filename=package://pnpush_config/models/IRB120/meshes/collision/link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 scale=0.0254 0.0254 0.0254; visual mesh filename=package://pnpush_config/models/IRB120/meshes/visual/link_2.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 scale=0.0254 0.0254 0.0254
- link link_3: geometry collision mesh filename=package://pnpush_config/models/IRB120/meshes/collision/link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 scale=0.0254 0.0254 0.0254; visual mesh filename=package://pnpush_config/models/IRB120/meshes/visual/link_3.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 scale=0.0254 0.0254 0.0254
- link link_4: geometry collision mesh filename=package://pnpush_config/models/IRB120/meshes/collision/link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 scale=0.0254 0.0254 0.0254; visual mesh filename=package://pnpush_config/models/IRB120/meshes/visual/link_4.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 scale=0.0254 0.0254 0.0254
- link link_5: geometry collision mesh filename=package://pnpush_config/models/IRB120/meshes/collision/link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 scale=0.0254 0.0254 0.0254; visual mesh filename=package://pnpush_config/models/IRB120/meshes/visual/link_5.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 scale=0.0254 0.0254 0.0254
- link link_6: geometry collision mesh filename=package://pnpush_config/models/IRB120/meshes/collision/link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 scale=0.0254 0.0254 0.0254; visual mesh filename=package://pnpush_config/models/IRB120/meshes/visual/link_6.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 scale=0.0254 0.0254 0.0254

Commit message: add moveit config for irb120

File: catkin_ws/src/pnpush_config/models/IRB120/irb_120.urdf (robot description, URDF)
Before this commit: robot irb_120, 7 links, 6 joints
Joints:
- joint joint1: origin xyz=0 0 0 rpy=-3.14159265359 3.14159265359 3.14159265359 -> xyz=0 0 0 rpy=-1.57079632679 3.14159265359 3.14159265359

File: catkin_ws/src/pnpush_config/models/IRB120/irb_120_drake.urdf (robot description, URDF)
Before this commit: robot irb_120, 7 links, 6 joints
Joints:
- joint joint1: origin xyz=0 0 0 rpy=-3.14159265359 3.14159265359 3.14159265359 -> xyz=0 0 0 rpy=-1.57079632679 3.14159265359 3.14159265359

Commit message: update irb120 urdf

File: catkin_ws/src/pnpush_config/models/IRB120/irb_120.urdf (robot description, URDF)
Before this commit: robot irb_120, 7 links, 6 joints
Links:
- added link link_ft; collision cylinder length=0.04 radius=0.037; visual cylinder length=0.04 radius=0.037
- added link link_probe; collision cylinder length=0.8673 radius=0.00789; visual cylinder length=0.08673 radius=0.00789
Joints:
- added joint joint7: type fixed, parent link_6, child link_ft, origin xyz=0 0 0.04 rpy=0 0 0, axis 0 0 1
- added joint joint8: type fixed, parent link_ft, child link_probe, origin xyz=0 0 0.08673  rpy=0 0 0, axis 0 0 1

File: catkin_ws/src/pnpush_config/models/IRB120/irb_120_drake.urdf (robot description, URDF)
Before this commit: robot irb_120, 7 links, 6 joints
Links:
- link base_link: geometry collision mesh filename=meshes/collision/base_link.stl scale=0.0254 0.0254 0.0254; visual mesh filename=meshes/visual/base_link.stl scale=0.0254 0.0254 0.0254
- link link_1: geometry collision mesh filename=meshes/collision/link_1.stl scale=0.0254 0.0254 0.0254; visual mesh filename=meshes/visual/link_1.stl scale=0.0254 0.0254 0.0254
- link link_2: geometry collision mesh filename=meshes/collision/link_2.stl scale=0.0254 0.0254 0.0254; visual mesh filename=meshes/visual/link_2.stl scale=0.0254 0.0254 0.0254
- link link_3: geometry collision mesh filename=meshes/collision/link_3.stl scale=0.0254 0.0254 0.0254; visual mesh filename=meshes/visual/link_3.stl scale=0.0254 0.0254 0.0254
- link link_4: geometry collision mesh filename=meshes/collision/link_4.stl scale=0.0254 0.0254 0.0254; visual mesh filename=meshes/visual/link_4.stl scale=0.0254 0.0254 0.0254
- link link_5: geometry collision mesh filename=meshes/collision/link_5.stl scale=0.0254 0.0254 0.0254; visual mesh filename=meshes/visual/link_5.stl scale=0.0254 0.0254 0.0254
- link link_6: geometry collision mesh filename=meshes/collision/link_6.stl scale=0.0254 0.0254 0.0254; visual mesh filename=meshes/visual/link_6.stl scale=0.0254 0.0254 0.0254

Commit message: using the probe 2

File: catkin_ws/src/pnpush_config/models/IRB120/irb_120.urdf (robot description, URDF)
Before this commit: robot irb_120, 9 links, 8 joints
Links:
- link link_probe: geometry collision cylinder length=0.16649 radius=0.004745; visual cylinder length=0.16649 radius=0.004745
Joints:
- joint joint8: origin xyz=0 0 0.23746 rpy=0 0 0 -> xyz=0 0 0.16649 rpy=0 0 0

Commit message: update to probe 3

File: catkin_ws/src/pnpush_config/models/IRB120/irb_120.urdf (robot description, URDF)
Before this commit: robot irb_120, 9 links, 8 joints
Links:
- link link_probe: geometry collision cylinder length=0.15947 radius=0.00475; visual cylinder length=0.15947 radius=0.00475
Joints:
- joint joint8: origin xyz=0 0 0.16649 rpy=0 0 0 -> xyz=0 0 0.15947 rpy=0 0 0

Commit message: Update irb_120.urdf

File: catkin_ws/src/pnpush_config/models/IRB120/irb_120.urdf (robot description, URDF)
Before this commit: robot irb_120, 9 links, 8 joints
Links:
- link link_probe: geometry collision cylinder length=0.15653 radius=0.00475; visual cylinder length=0.15653 radius=0.00475
Joints:
- joint joint8: origin xyz=0 0 0.15947 rpy=0 0 0 -> xyz=0 0 0.15653 rpy=0 0 0
